Commit message: added missing prefix to links (batch replace)

File: motoman_config/cfg/mh5_mesh_macro.xacro (robot description, xacro)
@@ -118,6 +118,6 @@
 		<!-- joint list -->
 		<joint name="${prefix}joint_s" type="revolute">
-			<parent link="base_link"/>
-			<child link="link_s"/>
+			<parent link="${prefix}base_link"/>
+			<child link="${prefix}link_s"/>
 			<origin xyz="0 0 0.1990" rpy="0 0 0"/>
 			<axis xyz="0 0 1" />
@@ -125,6 +125,6 @@
 		</joint>
 		<joint name="${prefix}joint_l" type="revolute">
-			<parent link="link_s"/>
-			<child link="link_l"/>
+			<parent link="${prefix}link_s"/>
+			<child link="${prefix}link_l"/>
 			<origin xyz="0.0880 0 0.1310" rpy="0 0 0"/>
 			<axis xyz="0 1 0" />
@@ -132,6 +132,6 @@
 		</joint>
 		<joint name="${prefix}joint_u" type="revolute">
-			<parent link="link_l"/>
-			<child link="link_u"/>
+			<parent link="${prefix}link_l"/>
+			<child link="${prefix}link_u"/>
 			<origin xyz="0 0 0.3100" rpy="0 0 0"/>
 			<axis xyz="0 -1 0" />
@@ -139,6 +139,6 @@
 		</joint>
 		<joint name="${prefix}joint_r" type="revolute">
-			<parent link="link_u"/>
-			<child link="link_r"/>
+			<parent link="${prefix}link_u"/>
+			<child link="${prefix}link_r"/>
 			<origin xyz="0.0715 0 0.0399" rpy="0 0 0"/>
 			<axis xyz="-1 0 0" />
@@ -146,6 +146,6 @@
 		</joint>
 		<joint name="${prefix}joint_b" type="revolute">
-			<parent link="link_r"/>
-			<child link="link_b"/>
+			<parent link="${prefix}link_r"/>
+			<child link="${prefix}link_b"/>
 			<origin xyz="0.2335 0 0" rpy="0 0 0"/>
 			<axis xyz="0 -1 0" />
@@ -153,6 +153,6 @@
 		</joint>
 		<joint name="${prefix}joint_t" type="revolute">
-			<parent link="link_b"/>
-			<child link="link_t"/>
+			<parent link="${prefix}link_b"/>
+			<child link="${prefix}link_t"/>
 			<origin xyz="0.0510 0 0" rpy="0 0 0"/>
 			<axis xyz="-1 0 0" />

File: motoman_config/cfg/sia10d_mesh_macro.xacro (robot description, xacro)
@@ -134,6 +134,6 @@
 		<!-- joint list -->
 		<joint name="${prefix}joint_s" type="revolute">
-			<parent link="base_link"/>
-			<child link="link_s"/>
+			<parent link="${prefix}base_link"/>
+			<child link="${prefix}link_s"/>
 			<origin xyz="0 0 0.36" rpy="0 0 0"/>
 			<axis xyz="0 0 1" />
@@ -141,6 +141,6 @@
 		</joint>
 		<joint name="${prefix}joint_l" type="revolute">
-			<parent link="link_s"/>
-			<child link="link_l"/>
+			<parent link="${prefix}link_s"/>
+			<child link="${prefix}link_l"/>
 			<origin xyz="0 0 0" rpy="0 0 0"/>
 			<axis xyz="0 1 0" />
@@ -148,6 +148,6 @@
 		</joint>
 		<joint name="${prefix}joint_e" type="revolute">
-			<parent link="link_l"/>
-			<child link="link_e"/>
+			<parent link="${prefix}link_l"/>
+			<child link="${prefix}link_e"/>
 			<origin xyz="0 0 0.36" rpy="0 0 0"/>
 			<axis xyz="0 0 1" />
@@ -155,6 +155,6 @@
 		</joint>
 		<joint name="${prefix}joint_u" type="revolute">
-			<parent link="link_e"/>
-			<child link="link_u"/>
+			<parent link="${prefix}link_e"/>
+			<child link="${prefix}link_u"/>
 			<origin xyz="0 0 0" rpy="0 0 0"/>
 			<axis xyz="0 -1 0" />
@@ -162,6 +162,6 @@
 		</joint>
 		<joint name="${prefix}joint_r" type="revolute">
-			<parent link="link_u"/>
-			<child link="link_r"/>
+			<parent link="${prefix}link_u"/>
+			<child link="${prefix}link_r"/>
 			<origin xyz="0 0 0.360" rpy="0 0 0"/>
 			<axis xyz="0 0 -1" />
@@ -169,6 +169,6 @@
 		</joint>
 		<joint name="${prefix}joint_b" type="revolute">
-			<parent link="link_r"/>
-			<child link="link_b"/>
+			<parent link="${prefix}link_r"/>
+			<child link="${prefix}link_b"/>
 			<origin xyz="0 0 0" rpy="0 0 0"/>
 			<axis xyz="0 -1 0" />
@@ -176,6 +176,6 @@
 		</joint>
 		<joint name="${prefix}joint_t" type="revolute">
-			<parent link="link_b"/>
-			<child link="link_t"/>
+			<parent link="${prefix}link_b"/>
+			<child link="${prefix}link_t"/>
 			<origin xyz="0 0 0.155" rpy="0 0 0"/>
 			<axis xyz="0 0 -1" />
